File: SIPM.kicad_pcb (KiCad board)
At the start: 2 copper layers, 50 parts, among them J1 Conn_01x13_Male, J2 Conn_ARM_JTAG_SWD_10, SW1 SW_Push, U1 STM32L432KBUx, U2 TLV1117-33IDCY, U3 MAX5026, U4 OPA196xDBV, U5 INA168, U6 OPA340UA, U7 LM7705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

Commit message: Add files via upload
Connections:
- net /ANALOG_T renamed ANALOG_T
- net /BIAS renamed BIAS
- net /BIAS/GNDlower renamed GNDboljse
- net /BIAS/MAX32V renamed MAX32V
- net /CURRENT renamed TOK_BRANJE
- net /DAC renamed DAC
- net /DIGITAL_T renamed DIGITAL_T
- net /NRST renamed NRST
- net /NTC renamed NTC
- net /SCL renamed SCL
- net /SDA renamed SDA
- net /SWDCLK renamed SWDCLK
- net /SWDIO renamed SWDIO
- net /SWO renamed SWO
- net /microprocesor/NTC_CS renamed NTC_CS
- net /microprocesor/NTC_SCLK renamed NTC_SCLK
- net /microprocesor/NTC_SO renamed NTC_SO
Routing:
- net GND: track 330.9 -> 273.5 mm
- net +3V3: track 226.1 -> 214.5 mm
- net GNDboljse: track 59.0 -> 52.6 mm
- net +5V: track 123.4 -> 119.8 mm
- net NTC_SCLK: track 34.6 -> 35.5 mm
- net NTC_CS: track 27.3 -> 27.9 mm
Other:
- net class Default: trace_width 0.5 -> 0.2
