File: mikroprocesor.sch (KiCad schematic (older format))
At the start: 22 parts, among them SW1 SW_Push, U1 STM32L432KBUx, U2 TLV1117-33IDCY

Commit message: Add files via upload
Parts:
- added R15: R, Resistor_SMD:R_0805_2012Metric_Pad1.15x1.40mm_HandSolder, symbol Device:R
- added U8: MAX6682, MAX6682footprint:SOP65P490X110-8N, symbol Amplifier_Difference2:MAX6682
Connections:
- net +3V3: now also U8.8 (Vcc)
- net ANALOG: now also R7.1; no longer R7.2
- net GND: now also U8.4 (GND)
- net at U1.14 (PB0): now also C8.1, R7.2
- net NTC_SO: now reaches U1.21 (PA11)
- net NTC_SO: now also U8.6 (SO)
- net NTC_CS: now reaches U1.7 (PA1)
- net NTC_CS: now also U8.5 (CS)
- new net: R15.1, U8.2 (R+)
- new net: R15.2, U8.3 (R-)
- new net NTC_SCLK: U1.11 (PA5), U8.7 (SCK)
- no-connect marks 18 -> 16
Other:
- moved on the sheet: C1, C8, R1, R7
Changed lines of the file:
@@
 L Device:C C1
 U 1 1 61E80AF9
-P 1850 4800
-F 0 "C1" H 1965 4846 50  0000 L CNN
-F 1 "C" H 1965 4755 50  0000 L CNN
-F 2 "Capacitor_SMD:C_0805_2012Metric_Pad1.15x1.40mm_HandSolder" H 1888 4650 50  0001 C CNN
-F 3 "~" H 1850 4800 50  0001 C CNN
-	1    1850 4800
+P 850 4800
+F 0 "C1" H 965 4846 50  0000 L CNN
+F 1 "C" H 965 4755 50  0000 L CNN
+F 2 "Capacitor_SMD:C_0805_2012Metric_Pad1.15x1.40mm_HandSolder" H 888 4650 50  0001 C CNN
+F 3 "~" H 850 4800 50  0001 C CNN
+	1    850  4800
 	1    0    0    -1
 $EndComp
@@
 L Device:R R1
 U 1 1 61E8182F
-P 2250 4800
-F 0 "R1" H 2320 4846 50  0000 L CNN
-F 1 "R" H 2320 4755 50  0000 L CNN
-F 2 "Resistor_SMD:R_0805_2012Metric_Pad1.15x1.40mm_HandSolder" V 2180 4800 50  0001 C CNN
-F 3 "~" H 2250 4800 50  0001 C CNN
-	1    2250 4800
-	1    0    0    -1
-$EndComp
-Wire Wire Line
-	1850 4950 1850 5050
-Wire Wire Line
-	1850 5050 2250 5050
-Wire Wire Line
-	2250 4950 2250 5050
-Connection ~ 2250 5050
-Wire Wire Line
-	2250 5050 2500 5050
+P 1200 4800
+F 0 "R1" H 1270 4846 50  0000 L CNN
+F 1 "R" H 1270 4755 50  0000 L CNN
+F 2 "Resistor_SMD:R_0805_2012Metric_Pad1.15x1.40mm_HandSolder" V 1130 4800 50  0001 C CNN
+F 3 "~" H 1200 4800 50  0001 C CNN
+	1    1200 4800
+	1    0    0    -1
+$EndComp
+Wire Wire Line
+	850  4950 850  5050
+Wire Wire Line
+	1200 4950 1200 5050
 $Comp
 L power:GND #PWR010
 U 1 1 61E81A95
-P 1850 4550
-F 0 "#PWR010" H 1850 4300 50  0001 C CNN
-F 1 "GND" H 1855 4377 50  0000 C CNN
-F 2 "" H 1850 4550 50  0001 C CNN
-F 3 "" H 1850 4550 50  0001 C CNN
-	1    1850 4550
+P 850 4550
+F 0 "#PWR010" H 850 4300 50  0001 C CNN
+F 1 "GND" H 855 4377 50  0000 C CNN
+F 2 "" H 850 4550 50  0001 C CNN
+F 3 "" H 850 4550 50  0001 C CNN
+	1    850  4550
 	-1   0    0    1
 $EndComp
 Wire Wire Line
-	1850 4550 1850 4650
+	850  4550 850  4650
 $Comp
 L power:+3.3V #PWR013
 U 1 1 61E82007
-P 2250 4550
-F 0 "#PWR013" H 2250 4400 50  0001 C CNN
-F 1 "+3.3V" H 2265 4723 50  0000 C CNN
-F 2 "" H 2250 4550 50  0001 C CNN
-F 3 "" H 2250 4550 50  0001 C CNN
-	1    2250 4550
-	1    0    0    -1
-$EndComp
-Wire Wire Line
-	2250 4550 2250 4650
+P 1200 4550
+F 0 "#PWR013" H 1200 4400 50  0001 C CNN
+F 1 "+3.3V" H 1215 4723 50  0000 C CNN
+F 2 "" H 1200 4550 50  0001 C CNN
+F 3 "" H 1200 4550 50  0001 C CNN
+	1    1200 4550
+	1    0    0    -1
+$EndComp
+Wire Wire Line
+	1200 4550 1200 4650
 Wire Wire Line
 	1850 5250 2250 5250
@@
 Connection ~ 3700 2600
 NoConn ~ 4000 3700
-NoConn ~ 4000 3800
 NoConn ~ 4000 3900
 NoConn ~ 4000 4000
@@
 NoConn ~ 4000 4600
 NoConn ~ 4000 4700
-NoConn ~ 4000 4800
 NoConn ~ 4000 4900
 NoConn ~ 4000 5200
@@
 NoConn ~ 3000 4300
 NoConn ~ 3000 4400
-NoConn ~ 3000 4600
 NoConn ~ 3000 4700
 NoConn ~ 3000 4900
@@
 L Device:R R7
 U 1 1 61E985B4
-P 4650 4200
-F 0 "R7" V 4857 4200 50  0000 C CNN
-F 1 "R" V 4766 4200 50  0000 C CNN
-F 2 "Resistor_SMD:R_0805_2012Metric_Pad1.15x1.40mm_HandSolder" V 4580 4200 50  0001 C CNN
-F 3 "~" H 4650 4200 50  0001 C CNN
-	1    4650 4200
+P 2150 4700
+F 0 "R7" V 2357 4700 50  0000 C CNN
+F 1 "R" V 2266 4700 50  0000 C CNN
+F 2 "Resistor_SMD:R_0805_2012Metric_Pad1.15x1.40mm_HandSolder" V 2080 4700 50  0001 C CNN
+F 3 "~" H 2150 4700 50  0001 C CNN
+	1    2150 4700
 	0    -1   -1   0
 $EndComp
@@
 L Device:C C8
 U 1 1 61E9AEC5
-P 4350 3950
-F 0 "C8" H 4465 3996 50  0000 L CNN
-F 1 "C" H 4465 3905 50  0000 L CNN
-F 2 "Capacitor_SMD:C_0805_2012Metric_Pad1.15x1.40mm_HandSolder" H 4388 3800 50  0001 C CNN
-F 3 "~" H 4350 3950 50  0001 C CNN
-	1    4350 3950
+P 2400 4550
+F 0 "C8" H 2515 4596 50  0000 L CNN
+F 1 "C" H 2515 4505 50  0000 L CNN
+F 2 "Capacitor_SMD:C_0805_2012Metric_Pad1.15x1.40mm_HandSolder" H 2438 4400 50  0001 C CNN
+F 3 "~" H 2400 4550 50  0001 C CNN
+	1    2400 4550
 	-1   0    0    1
 $EndComp
@@
 L power:GND #PWR021
 U 1 1 61E9C47D
-P 4350 3750
-F 0 "#PWR021" H 4350 3500 50  0001 C CNN
-F 1 "GND" H 4355 3577 50  0000 C CNN
-F 2 "" H 4350 3750 50  0001 C CNN
-F 3 "" H 4350 3750 50  0001 C CNN
-	1    4350 3750
+P 2400 4350
+F 0 "#PWR021" H 2400 4100 50  0001 C CNN
+F 1 "GND" H 2405 4177 50  0000 C CNN
+F 2 "" H 2400 4350 50  0001 C CNN
+F 3 "" H 2400 4350 50  0001 C CNN
+	1    2400 4350
 	-1   0    0    1
 $EndComp
 Wire Wire Line
-	4900 4200 4800 4200
-Text GLabel 4900 4200 2    50   Input ~ 0
+	2400 4700 2300 4700
+Text GLabel 1850 4700 0    50   Input ~ 0
 ANALOG
-Wire Wire Line
-	1600 5050 1850 5050
-Connection ~ 1850 5050
-Text GLabel 1600 5050 0    50   Input ~ 0
+Text GLabel 700  5050 0    50   Input ~ 0
 SCL
 Wire Wire Line
@@
 SDA
 Wire Wire Line
-	4000 4200 4350 4200
-Wire Wire Line
-	4350 3750 4350 3800
-Wire Wire Line
-	4350 4100 4350 4200
-Connection ~ 4350 4200
-Wire Wire Line
-	4350 4200 4500 4200
+	2400 4350 2400 4400
+Wire Wire Line
+	1850 4700 2000 4700
 $Comp
 L Device:R R6
@@
 L power:+3.3V #PWR022
 U 1 1 61F05150
-P 4350 4700
-F 0 "#PWR022" H 4350 4550 50  0001 C CNN
-F 1 "+3.3V" H 4365 4873 50  0000 C CNN
-F 2 "" H 4350 4700 50  0001 C CNN
-F 3 "" H 4350 4700 50  0001 C CNN
-	1    4350 4700
+P 4350 4600
+F 0 "#PWR022" H 4350 4450 50  0001 C CNN
+F 1 "+3.3V" H 4365 4773 50  0000 C CNN
+F 2 "" H 4350 4600 50  0001 C CNN
+F 3 "" H 4350 4600 50  0001 C CNN
+	1    4350 4600
 	-1   0    0    1
 $EndComp
-Wire Wire Line
-	4350 4700 4350 4600
 Wire Wire Line
 	4000 4300 4350 4300
@@
 Text GLabel 4800 4300 2    50   Input ~ 0
 DIGITAL
-Wire Wire Line
-	4100 3800 4100 4100
-Wire Wire Line
-	4100 4100 4000 4100
-Text GLabel 4100 3800 2    50   Input ~ 0
+Text GLabel 4300 4000 2    50   Input ~ 0
 DAC
 Wire Wire Line
@@
 Text GLabel 1950 3700 0    50   Input ~ 0
 NRST
+Wire Wire Line
+	700  5050 850  5050
+Wire Wire Line
+	1200 5050 2500 5050
+Wire Wire Line
+	850  5050 1200 5050
+Connection ~ 850  5050
+Connection ~ 1200 5050
+Wire Wire Line
+	3000 4600 2650 4600
+Wire Wire Line
+	2650 4600 2650 4700
+Wire Wire Line
+	2650 4700 2400 4700
+Connection ~ 2400 4700
+Wire Wire Line
+	4200 4100 4200 4000
+Wire Wire Line
+	4200 4000 4300 4000
+Wire Wire Line
+	4000 4100 4200 4100
+Wire Wire Line
+	4300 4200 4000 4200
+Text GLabel 4300 4200 2    50   Input ~ 0
+NTC_SCLK
+Wire Wire Line
+	4300 3800 4000 3800
+Text GLabel 4300 3800 2    50   Input ~ 0
+NTC_CS
+Wire Wire Line
+	4450 4850 4150 4850
+Wire Wire Line
+	4150 4850 4150 4800
+Wire Wire Line
+	4150 4800 4000 4800
+Text GLabel 4450 4850 2    50   Input ~ 0
+NTC_SO
+$Comp
+L Amplifier_Difference2:MAX6682 U8
+U 1 1 61F21190
+P 7800 2200
+F 0 "U8" H 7825 2678 50  0000 C CNN
+F 1 "MAX6682" H 7825 2587 50  0000 C CNN
+F 2 "MAX6682footprint:SOP65P490X110-8N" H 7800 2200 50  0001 C CNN
+F 3 "" H 7800 2200 50  0001 C CNN
+	1    7800 2200
+	1    0    0    -1
+$EndComp
+NoConn ~ 8250 2050
+$Comp
+L Device:R R15
+U 1 1 61F239ED
+P 8500 2200
+F 0 "R15" H 8570 2246 50  0000 L CNN
+F 1 "R" H 8570 2155 50  0000 L CNN
+F 2 "Resistor_SMD:R_0805_2012Metric_Pad1.15x1.40mm_HandSolder" V 8430 2200 50  0001 C CNN
+F 3 "~" H 8500 2200 50  0001 C CNN
+	1    8500 2200
+	1    0    0    -1
+$EndComp
+Wire Wire Line
+	8500 2050 8500 1950
+Wire Wire Line
+	8500 1950 8350 1950
+Wire Wire Line
+	8350 1950 8350 2150
+Wire Wire Line
+	8350 2150 8250 2150
+Wire Wire Line
+	8250 2250 8350 2250
+Wire Wire Line
+	8350 2250 8350 2350
+Wire Wire Line
+	8350 2350 8500 2350
+$Comp
+L power:GND #PWR0101
+U 1 1 61F285E3
+P 8050 2500
+F 0 "#PWR0101" H 8050 2250 50  0001 C CNN
+F 1 "GND" H 8055 2327 50  0000 C CNN
+F 2 "" H 8050 2500 50  0001 C CNN
+F 3 "" H 8050 2500 50  0001 C CNN
+	1    8050 2500
+	1    0    0    -1
+$EndComp
+$Comp
+L power:+3.3V #PWR0102
+U 1 1 61F28643
+P 7550 1900
+F 0 "#PWR0102" H 7550 1750 50  0001 C CNN
+F 1 "+3.3V" H 7565 2073 50  0000 C CNN
+F 2 "" H 7550 1900 50  0001 C CNN
+F 3 "" H 7550 1900 50  0001 C CNN
+	1    7550 1900
+	1    0    0    -1
+$EndComp
+Wire Wire Line
+	7700 2550 7700 2500
+Text GLabel 7700 2550 3    50   Input ~ 0
+NTC_CS
+Wire Wire Line
+	7350 2350 7400 2350
+Text GLabel 7350 2350 0    50   Input ~ 0
+NTC_SO
+Wire Wire Line
+	7150 2200 7250 2200
+Wire Wire Line
+	7250 2200 7250 2250
+Wire Wire Line
+	7250 2250 7400 2250
+Text GLabel 7150 2200 0    50   Input ~ 0
+NTC_SCLK
 $EndSCHEMATC

Commit message: Add files via upload
Connections:
- net NTC: now reaches R15.2, U8.3 (R-)
Changed lines of the file:
@@
 Text GLabel 7150 2200 0    50   Input ~ 0
 NTC_SCLK
+Wire Wire Line
+	8500 2450 8500 2350
+Connection ~ 8500 2350
+Text GLabel 8500 2450 3    50   Input ~ 0
+NTC
 $EndSCHEMATC

Commit message: Add files via upload
Connections:
- net TOK_BRANJE: now reaches U1.8 (PA2)
- net ANALOG renamed ANALOG_T
- net DIGITAL renamed DIGITAL_T
- no-connect marks 16 -> 15
Changed lines of the file:
@@
 Connection ~ 3700 2600
 NoConn ~ 4000 3700
-NoConn ~ 4000 3900
 NoConn ~ 4000 4000
 NoConn ~ 4000 4400
@@
 Wire Wire Line
 	2400 4700 2300 4700
-Text GLabel 1850 4700 0    50   Input ~ 0
-ANALOG
 Text GLabel 700  5050 0    50   Input ~ 0
 SCL
@@
 	4800 4300 4350 4300
 Connection ~ 4350 4300
-Text GLabel 4800 4300 2    50   Input ~ 0
-DIGITAL
 Text GLabel 4300 4000 2    50   Input ~ 0
 DAC
@@
 Text GLabel 8500 2450 3    50   Input ~ 0
 NTC
+Wire Wire Line
+	4650 3900 4000 3900
+Text GLabel 4650 3900 2    50   Input ~ 0
+TOK_BRANJE
+Text GLabel 4800 4300 2    50   Input ~ 0
+DIGITAL_T
+Text GLabel 1850 4700 0    50   Input ~ 0
+ANALOG_T
 $EndSCHEMATC

Commit message: Add files via upload
Parts:
- L1: footprint (none) -> Inductor_SMD:L_0805_2012Metric_Pad1.15x1.40mm_HandSolder
- SW1: footprint (none) -> Button_Switch_SMD:SW_DIP_SPSTx02_Slide_6.7x6.64mm_W8.61mm_P2.54mm_LowProfile
Changed lines of the file:
@@
 F 0 "L1" V 4355 2650 50  0000 C CNN
 F 1 "L_Core_Ferrite_Small" V 4264 2650 50  0000 C CNN
-F 2 "" H 4150 2650 50  0001 C CNN
+F 2 "Inductor_SMD:L_0805_2012Metric_Pad1.15x1.40mm_HandSolder" H 4150 2650 50  0001 C CNN
 F 3 "~" H 4150 2650 50  0001 C CNN
 	1    4150 2650
@@
 F 0 "SW1" V 2246 3952 50  0000 R CNN
 F 1 "SW_Push" V 2155 3952 50  0000 R CNN
-F 2 "" H 2200 4200 50  0001 C CNN
+F 2 "Button_Switch_SMD:SW_DIP_SPSTx02_Slide_6.7x6.64mm_W8.61mm_P2.54mm_LowProfile" H 2200 4200 50  0001 C CNN
 F 3 "" H 2200 4200 50  0001 C CNN
 	1    2200 4000

Commit message: Add files via upload
Connections:
- net TOK_BRANJE renamed CURRENT
Changed lines of the file:
@@
 Wire Wire Line
 	2400 4700 2300 4700
-Text GLabel 700  5050 0    50   Input ~ 0
-SCL
 Wire Wire Line
 	1600 5250 1850 5250
 Connection ~ 1850 5250
-Text GLabel 1600 5250 0    50   Input ~ 0
-SDA
 Wire Wire Line
 	2400 4350 2400 4400
@@
 	4800 4300 4350 4300
 Connection ~ 4350 4300
-Text GLabel 4300 4000 2    50   Input ~ 0
-DAC
 Wire Wire Line
 	4300 5000 4000 5000
-Text GLabel 4300 5000 2    50   Input ~ 0
-SWDIO
 Wire Wire Line
 	4250 5100 4000 5100
-Text GLabel 4250 5100 2    50   Input ~ 0
-SWDCLK
-Text GLabel 3000 4800 0    50   Input ~ 0
-SWO
-Text GLabel 1950 3700 0    50   Input ~ 0
-NRST
 Wire Wire Line
 	700  5050 850  5050
@@
 Wire Wire Line
 	4300 4200 4000 4200
-Text GLabel 4300 4200 2    50   Input ~ 0
-NTC_SCLK
 Wire Wire Line
 	4300 3800 4000 3800
-Text GLabel 4300 3800 2    50   Input ~ 0
-NTC_CS
 Wire Wire Line
 	4450 4850 4150 4850
@@
 Wire Wire Line
 	4150 4800 4000 4800
-Text GLabel 4450 4850 2    50   Input ~ 0
-NTC_SO
 $Comp
 L Amplifier_Difference2:MAX6682 U8
@@
 Wire Wire Line
 	7700 2550 7700 2500
-Text GLabel 7700 2550 3    50   Input ~ 0
-NTC_CS
 Wire Wire Line
 	7350 2350 7400 2350
-Text GLabel 7350 2350 0    50   Input ~ 0
-NTC_SO
 Wire Wire Line
 	7150 2200 7250 2200
@@
 Wire Wire Line
 	7250 2250 7400 2250
-Text GLabel 7150 2200 0    50   Input ~ 0
-NTC_SCLK
 Wire Wire Line
 	8500 2450 8500 2350
 Connection ~ 8500 2350
-Text GLabel 8500 2450 3    50   Input ~ 0
-NTC
 Wire Wire Line
 	4650 3900 4000 3900
-Text GLabel 4650 3900 2    50   Input ~ 0
-TOK_BRANJE
-Text GLabel 4800 4300 2    50   Input ~ 0
+Text HLabel 8500 2450 3    50   Input ~ 0
+NTC
+Text Label 7150 2200 2    50   ~ 0
+NTC_SCLK
+Text Label 7350 2350 2    50   ~ 0
+NTC_SO
+Text Label 7700 2550 3    50   ~ 0
+NTC_CS
+Text Label 4300 3800 0    50   ~ 0
+NTC_CS
+Text HLabel 4650 3900 2    50   Input ~ 0
+CURRENT
+Text HLabel 4300 4000 2    50   Input ~ 0
+DAC
+Text Label 4300 4200 0    50   ~ 0
+NTC_SCLK
+Text HLabel 4800 4300 2    50   Input ~ 0
 DIGITAL_T
-Text GLabel 1850 4700 0    50   Input ~ 0
+Text Label 4450 4850 0    50   ~ 0
+NTC_SO
+Text HLabel 4300 5000 2    50   Input ~ 0
+SWDIO
+Text HLabel 4250 5100 2    50   Input ~ 0
+SWDCLK
+Text HLabel 1600 5250 0    50   Input ~ 0
+SDA
+Text HLabel 700  5050 0    50   Input ~ 0
+SCL
+Text HLabel 3000 4800 0    50   Input ~ 0
+SWO
+Text HLabel 1850 4700 0    50   Input ~ 0
 ANALOG_T
+Text HLabel 1950 3700 0    50   Input ~ 0
+NRST
 $EndSCHEMATC
