File: microprocesor.sch (KiCad schematic (older format))
At the start: 24 parts, among them SW1 SW_Push, U1 STM32L432KBUx, U2 TLV1117-33IDCY, U8 MAX6682

Commit message: Add files via upload
Parts:
- added C22: 100 nF, Capacitor_SMD:C_0805_2012Metric_Pad1.15x1.40mm_HandSolder, symbol Device:C
- C1, C2: value C -> 0 pF
- C10: value C -> 10 μF
- C11: value C -> 100 μF
- C3, C5, C6, C8: value C -> 100 nF
- C4: value C -> 4.7 μF
- C7: value C -> 10 nF
- C9: value C -> 1 μF
- R1, R2, R7: value R -> 10 kΩ
- R15: value R -> 3.915 kΩ
- R3: value R -> 470 Ω
- R4, R5: value R -> 100 Ω
- R6: value R -> 4.7 kΩ
- SW1: footprint Button_Switch_SMD:SW_DIP_SPSTx02_Slide_6.7x6.64mm_W8.61mm_P2.54mm_LowProfile -> gumbfootprint:430182050816
Connections:
- net GND: now also C22.1
- net +3V3 renamed +3.3V
- net +3.3V: now also C22.2

Commit message: Add files via upload
Parts:
- C11: footprint Capacitor_SMD:C_0805_2012Metric_Pad1.15x1.40mm_HandSolder -> 100ukondenzatorfootprint:CAPE830X690N
- R15: value 3.915 kΩ -> 3.9 kΩ
- U2: footprint TLV1117footprint:SOT230P700X180-4N -> TLV1117footprintm:TO228P970X238-3N
Connections:
- net +3.3V: no longer U2.4 (OUTPUT)
- no-connect marks 15 -> 16
Changed lines of the file:
@@
 F 0 "U2" H 8225 7465 50  0000 C CNN
 F 1 "TLV1117-33IDCY" H 8225 7374 50  0000 C CNN
-F 2 "TLV1117footprint:SOT230P700X180-4N" H 8200 6400 50  0001 C CNN
+F 2 "TLV1117footprintm:TO228P970X238-3N" H 8200 6400 50  0001 C CNN
 F 3 "" H 8200 6400 50  0001 C CNN
 	1    6800 5350
@@
 F 0 "C11" H 9815 4296 50  0000 L CNN
 F 1 "100 μF" H 9815 4205 50  0000 L CNN
-F 2 "Capacitor_SMD:C_0805_2012Metric_Pad1.15x1.40mm_HandSolder" H 9738 4100 50  0001 C CNN
+F 2 "100ukondenzatorfootprint:CAPE830X690N" H 9738 4100 50  0001 C CNN
 F 3 "~" H 9700 4250 50  0001 C CNN
 	1    9700 4250
@@
 Connection ~ 8200 5100
 Wire Wire Line
-	9200 3600 9400 3600
-Wire Wire Line
-	9400 3600 9400 3900
-Wire Wire Line
-	9400 3900 9200 3900
-Wire Wire Line
-	9400 3600 9700 3600
-Wire Wire Line
 	9700 3600 9700 4100
-Connection ~ 9400 3600
 Wire Wire Line
 	10100 3600 9700 3600
@@
 AR Path="/62053103/620536F3" Ref="R15"  Part="1"
 F 0 "R15" H 9120 1746 50  0000 L CNN
-F 1 "3.915 kΩ" H 9120 1655 50  0000 L CNN
+F 1 "3.9 kΩ" H 9120 1655 50  0000 L CNN
 F 2 "Resistor_SMD:R_0805_2012Metric_Pad1.15x1.40mm_HandSolder" V 8980 1700 50  0001 C CNN
 F 3 "~" H 9050 1700 50  0001 C CNN
@@
 Text HLabel 1400 4050 1    50   Input ~ 0
 GND
+NoConn ~ 9200 3900
+Wire Wire Line
+	9200 3600 9700 3600
 $EndSCHEMATC
