File: napetostSiPM.kicad_pcb (KiCad board)
At the start: 2 copper layers, 50 parts, among them J1 Conn_01x13_Male, J2 Conn_ARM_JTAG_SWD_10, SW1 SW_Push, U1 STM32L432KBUx, U2 TLV1117-33IDCY, U3 MAX5026, U4 OPA196xDBV, U5 INA168, U6 OPA340UA, U7 LM7705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

Commit message: Add files via upload
Parts:
- moved R10 9.06 mm to (148.8, 143.5), turned to 0 degrees
- moved C15 5.06 mm to (147.3, 134.6)
- moved U9 3.19 mm to (149.2, 139.1), turned to 270 degrees
- moved R13 1.29 mm to (149.9, 128.3)
- moved L2 0.64 mm to (154.9, 141.6), turned to 0 degrees
- moved R11 0.22 mm to (149.9, 130.8)
Routing:
- net Net-(R10-Pad2): track 6.07 -> 15.3 mm, vias 0 -> 2
- net Net-(L2-Pad1): track 16.4 -> 7.32 mm
- net +3V3: track 226.1 -> 233.2 mm
- net Net-(C15-Pad1): track 22.5 -> 18.2 mm
- net GND: track 330.9 -> 332.8 mm
- net /BIAS/MAX32V: track 15.7 -> 14.9 mm
- net +5V: track 123.4 -> 123.3 mm, vias 0 -> 2
Other:
- net class Default: trace_width 0.5 -> 0.2

Commit message: Add files via upload
Parts:
- added C22: 100 nF, Capacitor_SMD:C_0805_2012Metric_Pad1.15x1.40mm_HandSolder, F.Cu at (185.4, 127.2)
- added C23: 10 nF, Capacitor_SMD:C_0805_2012Metric_Pad1.15x1.40mm_HandSolder, F.Cu at (157.3, 123.2)
- C1, C2: value C -> 0 pF
- C10: value C -> 10 μF
- C11: value C -> 100 μF
- C12, C4: value C -> 4.7 μF
- C13, C14, C17, C18, C3, C5, C6, C8: value C -> 100 nF
- C15, C16, C9: value C -> 1 μF
- C19, C21: value C -> 22 μF
- C20: value C -> 5 μF
- C7: value C -> 10 nF
- L2: value L -> 47 μH; footprint A915BY-470Mfootprint:IND_#A915BY-470M=P3 -> tuljavafootprint:Wurth_Electronics-74451147-Manufacturer_Recommended
- R1, R2, R7, R8: value R -> 10 kΩ
- R10: value R -> 1156 kΩ
- R11: value R -> 47 kΩ
- R12: value R -> 5 Ω
- R13, R4, R5: value R -> 100 Ω
- R14: value R -> 500 kΩ
- R15: value R -> 3.915 kΩ
- R3: value R -> 470 Ω
- R6: value R -> 4.7 kΩ
- R9: value R -> 100 kΩ
- SW1: footprint Button_Switch_SMD:SW_DIP_SPSTx02_Slide_6.7x6.64mm_W8.61mm_P2.54mm_LowProfile -> gumbfootprint:430182050816
- moved R12 2.78 mm to (167.6, 122.9)
- moved R14 2.77 mm to (160.0, 123.2)
- moved U5 2.69 mm to (163.8, 122.9)
- moved R15 0.73 mm to (182.6, 121.9)
- moved SW1 0.65 mm to (165.7, 150.5)
- moved C17 0.53 mm to (161.5, 119.4)
Connections:
- net +3V3 renamed /+3.3V
- net +5V renamed /+5V
- net GND renamed /GND
Routing:
- net /GND: track 332.8 -> 346.3 mm, vias 6 -> 9
- net Net-(C23-Pad2): track 7.31 -> 10.2 mm
- net /+3.3V: track 233.2 -> 235.2 mm
- net /+5V: track 123.3 -> 124.5 mm
- net Net-(R15-Pad1): track 3.20 -> 4.28 mm
- net /BIAS: track 33.7 -> 34.6 mm, vias 3 -> 2
- added copper zone on B.Cu, net /GND
- added copper zone on F.Cu, net /GND
Other:
- board outline added: 49.5 x 40.6 mm
- board text added: "E.S., M.V. @JSI 2022, v.01"

Commit message: Add files via upload
Parts:
- removed C19, C21: 22 μF, Capacitor_SMD:C_0805_2012Metric_Pad1.15x1.40mm_HandSolder
- removed C20: 5 μF, Capacitor_SMD:C_0805_2012Metric_Pad1.15x1.40mm_HandSolder
- removed U7: LM7705, LM7705footprint:SOP65P490X110-8N
- C11: footprint Capacitor_SMD:C_0805_2012Metric_Pad1.15x1.40mm_HandSolder -> 100ukondenzatorfootprint:CAPE830X690N
- R10: value 1156 kΩ -> 1.2 MΩ
- R12: value 5 Ω -> 4.7 Ω
- R14: value 500 kΩ -> 470 kΩ
- R15: value 3.915 kΩ -> 3.9 kΩ
- U2: footprint TLV1117footprint:SOT230P700X180-4N -> TLV1117footprintm:TO228P970X238-3N
- U4: footprint OPA196xDBVfootprint:SOT95P280X145-5N -> Package_SO:VSSOP-8_3.0x3.0mm_P0.65mm
- U5: footprint Package_TO_SOT_SMD:SOT-23-5 -> Package_SO:TSSOP-8_4.4x3mm_P0.65mm
- U9: footprint diodafootprint:SOT91P240X105-3N -> diodafootprint:SOT-23-dioda
- moved SW1 3.36 mm to (164.6, 153.7)
- moved R12 3.18 mm to (170.8, 122.9)
- moved R8 2.86 mm to (157.5, 133.3), turned to 90 degrees
- moved C11 2.19 mm to (163.0, 145.4), turned to 180 degrees
- moved R10 1.94 mm to (149.2, 141.6)
- moved U5 1.58 mm to (165.3, 122.9), turned to 180 degrees
- moved C14 1.55 mm to (167.6, 127.4)
- moved R9 1.55 mm to (165.1, 127.4)
- moved U2 1.41 mm to (163.8, 137.2)
- moved L2 1.27 mm to (154.9, 140.3)
- moved C13 0.64 mm to (155.6, 128.3)
- moved U4 0.64 mm to (160.0, 127.6)
- moved R3 0.63 mm to (170.4, 144.1)
- moved U9 0.50 mm to (148.8, 138.8)
Connections:
- C13 pad 2: /BIAS/GNDlower -> /GND
- C17 pad 1: /+5V -> /+3.3V
- C18 pad 1: /+5V -> /+3.3V
- C18 pad 2: /BIAS/GNDlower -> /GND
- R12 pad 1: Net-(C14-Pad1) -> /BIAS
- R12 pad 2: /BIAS -> Net-(C14-Pad1)
- U4 pad 1: Net-(C14-Pad1) -> Net-(U4-Pad1)
- U4 pad 2: /BIAS/GNDlower -> Net-(C14-Pad2)
- U4 pad 4: Net-(C14-Pad2) -> /GND
- U4 pad 5: /BIAS/MAX32V -> Net-(U4-Pad5)
- U5 pad 1: Net-(C23-Pad2) -> /BIAS
- U5 pad 2: /GND -> Net-(C14-Pad1)
- U5 pad 3: Net-(C14-Pad1) -> Net-(U5-Pad3)
- U5 pad 4: /BIAS -> /GND
- U5 pad 5: /+5V -> Net-(U5-Pad5)
- U6 pad 4: /BIAS/GNDlower -> /GND
- U6 pad 7: /+5V -> /+3.3V
Routing:
- net /BIAS/GNDlower: track 59.1 -> 0.00 mm, vias 3 -> 0
- net /+3.3V: track 235.2 -> 286.1 mm, vias 7 -> 10
- net /+5V: track 124.5 -> 90.1 mm
- net /GND: track 346.3 -> 379.9 mm, vias 9 -> 14
- net Net-(C14-Pad2): track 7.99 -> 17.8 mm
- net /BIAS: track 34.6 -> 26.5 mm
- net Net-(C20-Pad1): track 3.73 -> 0.00 mm
- net Net-(C21-Pad2): track 3.59 -> 0.00 mm
- net Net-(C20-Pad2): track 2.88 -> 0.00 mm
- net Net-(R10-Pad2): track 15.3 -> 18.1 mm
- net /BIAS/MAX32V: track 14.9 -> 17.7 mm
- net /DAC: track 31.9 -> 33.7 mm
- net /NRST: track 25.6 -> 23.9 mm
- net Net-(C15-Pad1): track 18.2 -> 17.0 mm
- net Net-(C14-Pad1): track 15.4 -> 14.8 mm
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- removed copper zone on B.Cu, net /GND
- removed copper zone on F.Cu, net /GND
Other:
- board text added: "E.S., M.V. @JSI 2022, v.02"
- board text removed: "E.S., M.V. @JSI 2022, v.01"
