File: napetostSiPM.sch (KiCad schematic (older format))
At the start: 24 parts, among them U1 AD8001AN, U2 MAX5026, U3 INA168, U4 AD8001AN, U5 LM7705

Commit message: Add files via upload
Parts:
- removed C1, C10, C2, C3, C4, C5, C6, C7, C8, C9: C, Capacitor_SMD:C_0805_2012Metric_Pad1.15x1.40mm_HandSolder, symbol Device:C
- removed D1: D_Schottky, symbol Device:D_Schottky
- removed L1: L, symbol Device:L
- removed R1, R2, R3, R4, R5, R6, R7: R, Resistor_SMD:R_0805_2012Metric_Pad1.15x1.40mm_HandSolder, symbol Device:R
- removed U1, U4: AD8001AN, Package_DIP:DIP-8_W7.62mm, symbol Amplifier_Operational:AD8001AN
- removed U2: MAX5026, MAX5026footprint:SOT95P280X145-6N, symbol Amplifier_Difference:MAX5026
- removed U3: INA168, Package_TO_SOT_SMD:SOT-23-5, symbol Amplifier_Current:INA168
- removed U5: LM7705, LM7705footprint:SOP65P490X110-8N, symbol Amplifier_Difference:LM7705
- added J1: Conn_01x14_Male, symbol Connector:Conn_01x14_Male
- added J2: Conn_ARM_JTAG_SWD_10, Connector_PinHeader_1.27mm:PinHeader_2x05_P1.27mm_Vertical_SMD, symbol Connector:Conn_ARM_JTAG_SWD_10
Connections:
- net labels added: +3.3V, ANALOG, BIAS, BRANJE, DIGITAL, NRST, SCL, SDA, SWDCLK, SWDIO, SWO
- net labels removed: GNDboljse, MAX:32V
- wire segments 97 -> 18
- no-connect marks 0 -> 1

Commit message: Add files via upload
Parts:
- removed J1: Conn_01x14_Male, symbol Connector:Conn_01x14_Male
- added J1: Conn_01x13_Male, symbol Connector:Conn_01x13_Male
Connections:
- net labels added: NTC
- wire segments 18 -> 17
Changed lines of the file:
@@
 Wire Wire Line
 	8800 2650 8250 2650
-Text GLabel 8800 2750 2    50   Input ~ 0
+Text GLabel 8800 2550 2    50   Input ~ 0
 SCL
-Text GLabel 8800 2850 2    50   Input ~ 0
+Text GLabel 8800 2650 2    50   Input ~ 0
 SDA
 Wire Wire Line
@@
 SWO
 $Comp
-L Connector:Conn_01x14_Male J1
-U 1 1 61F59C6C
+L Connector:Conn_01x13_Male J1
+U 1 1 61EE8518
 P 8050 2150
 F 0 "J1" H 8156 2928 50  0000 C CNN
-F 1 "Conn_01x14_Male" H 8156 2837 50  0000 C CNN
+F 1 "Conn_01x13_Male" H 8156 2837 50  0000 C CNN
 F 2 "" H 8050 2150 50  0001 C CNN
 F 3 "~" H 8050 2150 50  0001 C CNN
@@
 $EndComp
 Wire Wire Line
-	8250 2750 8800 2750
-Wire Wire Line
-	8250 2850 8800 2850
-$Comp
-L power:+3.3V #PWR0101
-U 1 1 61F5A467
-P 8800 2550
-F 0 "#PWR0101" H 8800 2400 50  0001 C CNN
-F 1 "+3.3V" V 8815 2678 50  0000 L CNN
-F 2 "" H 8800 2550 50  0001 C CNN
-F 3 "" H 8800 2550 50  0001 C CNN
-	1    8800 2550
-	0    1    1    0
-$EndComp
-$Comp
-L power:GND #PWR0102
-U 1 1 61F5A61E
-P 8800 2650
-F 0 "#PWR0102" H 8800 2400 50  0001 C CNN
-F 1 "GND" V 8805 2522 50  0000 R CNN
-F 2 "" H 8800 2650 50  0001 C CNN
-F 3 "" H 8800 2650 50  0001 C CNN
-	1    8800 2650
-	0    -1   -1   0
-$EndComp
+	8600 2750 8250 2750
+Text GLabel 8600 2750 2    50   Input ~ 0
+NTC
 $EndSCHEMATC

Commit message: Add files via upload
Parts:
- removed J1: Conn_01x13_Male, symbol Connector:Conn_01x13_Male
- added J?: Conn_01x13_Male, symbol Connector:Conn_01x13_Male
Connections:
- net +3V3: now also J?.8 (Pin_8)
- net +5V: now also J?.3 (Pin_3)
- net BIAS: now also J?.5 (Pin_5)
- net GND: now also J?.1 (Pin_1), J?.13 (Pin_13), J?.2 (Pin_2), J?.4 (Pin_4), J?.9 (Pin_9)
- net NTC: now also J?.12 (Pin_12)
- net SCL: now also J?.10 (Pin_10)
- net SDA: now also J?.11 (Pin_11)
- new net ANALOG_T: J?.6 (Pin_6)
- new net DIGITAL_T: J?.7 (Pin_7)
Changed lines of the file:
@@
 	8800 1950 8250 1950
 Wire Wire Line
-	8500 2050 8250 2050
+	8950 2050 8250 2050
 Wire Wire Line
-	8950 2150 8250 2150
-Text GLabel 8950 2150 2    50   Input ~ 0
-ANALOG
-Wire Wire Line
-	8550 2350 8250 2350
+	8550 2250 8250 2250
 $Comp
 L power:+3.3V #PWR06
 U 1 1 61EC92B3
-P 8550 2350
-F 0 "#PWR06" H 8550 2200 50  0001 C CNN
-F 1 "+3.3V" V 8565 2478 50  0000 L CNN
-F 2 "" H 8550 2350 50  0001 C CNN
-F 3 "" H 8550 2350 50  0001 C CNN
-	1    8550 2350
+P 8550 2250
+F 0 "#PWR06" H 8550 2100 50  0001 C CNN
+F 1 "+3.3V" V 8565 2378 50  0000 L CNN
+F 2 "" H 8550 2250 50  0001 C CNN
+F 3 "" H 8550 2250 50  0001 C CNN
+	1    8550 2250
 	0    1    1    0
 $EndComp
 Wire Wire Line
-	8350 2450 8250 2450
+	8350 2350 8250 2350
 $Comp
 L power:GND #PWR01
 U 1 1 61ED4863
-P 8350 2450
-F 0 "#PWR01" H 8350 2200 50  0001 C CNN
-F 1 "GND" V 8355 2322 50  0000 R CNN
-F 2 "" H 8350 2450 50  0001 C CNN
-F 3 "" H 8350 2450 50  0001 C CNN
-	1    8350 2450
+P 8350 2350
+F 0 "#PWR01" H 8350 2100 50  0001 C CNN
+F 1 "GND" V 8355 2222 50  0000 R CNN
+F 2 "" H 8350 2350 50  0001 C CNN
+F 3 "" H 8350 2350 50  0001 C CNN
+	1    8350 2350
 	0    -1   -1   0
 $EndComp
 Wire Wire Line
+	8800 2450 8250 2450
+Wire Wire Line
 	8800 2550 8250 2550
-Wire Wire Line
-	8800 2650 8250 2650
+Text GLabel 8800 2450 2    50   Input ~ 0
+SCL
 Text GLabel 8800 2550 2    50   Input ~ 0
-SCL
-Text GLabel 8800 2650 2    50   Input ~ 0
 SDA
 Wire Wire Line
-	8550 2250 8250 2250
-Text GLabel 8550 2250 2    50   Input ~ 0
-DIGITAL
+	8550 2150 8250 2150
 $Comp
 L Connector:Conn_ARM_JTAG_SWD_10 J?
@@
 Text GLabel 8800 1950 2    50   Input ~ 0
 BIAS
-Text GLabel 8500 2050 2    50   Input ~ 0
-BRANJE
 Text GLabel 9050 4300 2    50   Input ~ 0
 NRST
@@
 Text GLabel 9050 4700 2    50   Input ~ 0
 SWO
+Wire Wire Line
+	8600 2650 8250 2650
+Text GLabel 8600 2650 2    50   Input ~ 0
+NTC
+Wire Wire Line
+	8400 2750 8250 2750
 $Comp
-L Connector:Conn_01x13_Male J1
-U 1 1 61EE8518
+L power:GND #PWR0103
+U 1 1 61EFC12A
+P 8400 2750
+F 0 "#PWR0103" H 8400 2500 50  0001 C CNN
+F 1 "GND" V 8405 2622 50  0000 R CNN
+F 2 "" H 8400 2750 50  0001 C CNN
+F 3 "" H 8400 2750 50  0001 C CNN
+	1    8400 2750
+	0    -1   -1   0
+$EndComp
+$Comp
+L Connector:Conn_01x13_Male J?
+U 1 1 61F8017B
 P 8050 2150
-F 0 "J1" H 8156 2928 50  0000 C CNN
+F 0 "J?" H 8156 2928 50  0000 C CNN
 F 1 "Conn_01x13_Male" H 8156 2837 50  0000 C CNN
 F 2 "" H 8050 2150 50  0001 C CNN
@@
 	1    0    0    -1
 $EndComp
-Wire Wire Line
-	8600 2750 8250 2750
-Text GLabel 8600 2750 2    50   Input ~ 0
-NTC
+Text GLabel 8950 2050 2    50   Input ~ 0
+ANALOG_T
+Text GLabel 8550 2150 2    50   Input ~ 0
+DIGITAL_T
 $EndSCHEMATC

Commit message: Add files via upload
Parts:
- J1: renamed from J?; footprint (none) -> Connector_PinHeader_2.54mm:PinHeader_1x13_P2.54mm_Vertical
Changed lines of the file:
@@
 $EndComp
 $Comp
-L Connector:Conn_01x13_Male J?
+L Connector:Conn_01x13_Male J1
 U 1 1 61F8017B
 P 8050 2150
-F 0 "J?" H 8156 2928 50  0000 C CNN
+F 0 "J1" H 8156 2928 50  0000 C CNN
 F 1 "Conn_01x13_Male" H 8156 2837 50  0000 C CNN
-F 2 "" H 8050 2150 50  0001 C CNN
+F 2 "Connector_PinHeader_2.54mm:PinHeader_1x13_P2.54mm_Vertical" H 8050 2150 50  0001 C CNN
 F 3 "~" H 8050 2150 50  0001 C CNN
 	1    8050 2150

Commit message: Add files via upload
Changed lines of the file:
@@
 Comment4 ""
 $EndDescr
-$Sheet
-S 2250 1500 1650 900
-U 61E803D7
-F0 "mikroprocesor" 50
-F1 "mikroprocesor.sch" 50
-$EndSheet
 $Comp
 L power:GND #PWR02
@@
 Wire Wire Line
 	8800 2550 8250 2550
-Text GLabel 8800 2450 2    50   Input ~ 0
-SCL
-Text GLabel 8800 2550 2    50   Input ~ 0
-SDA
 Wire Wire Line
 	8550 2150 8250 2150
@@
 	8550 3800 8550 4000
 NoConn ~ 9050 4800
-$Sheet
-S 1800 3900 2650 1050
-U 61F20E3B
-F0 "delanjeBIAS" 50
-F1 "delanjeBIAS.sch" 50
-$EndSheet
-Text GLabel 8800 1950 2    50   Input ~ 0
-BIAS
-Text GLabel 9050 4300 2    50   Input ~ 0
-NRST
-Text GLabel 9050 4500 2    50   Input ~ 0
-SWDCLK
-Text GLabel 9050 4600 2    50   Input ~ 0
-SWDIO
-Text GLabel 9050 4700 2    50   Input ~ 0
-SWO
 Wire Wire Line
 	8600 2650 8250 2650
-Text GLabel 8600 2650 2    50   Input ~ 0
-NTC
 Wire Wire Line
 	8400 2750 8250 2750
@@
 	1    0    0    -1
 $EndComp
-Text GLabel 8950 2050 2    50   Input ~ 0
+Text Label 8800 1950 0    50   ~ 0
+BIAS
+Text Label 8950 2050 0    50   ~ 0
 ANALOG_T
-Text GLabel 8550 2150 2    50   Input ~ 0
+Text Label 8550 2150 0    50   ~ 0
 DIGITAL_T
+Text Label 8800 2450 0    50   ~ 0
+SCL
+Text Label 8800 2550 0    50   ~ 0
+SDA
+Text Label 8600 2650 0    50   ~ 0
+NTC
+Text Label 9050 4300 0    50   ~ 0
+NRST
+Text Label 9050 4500 0    50   ~ 0
+SWDCLK
+Text Label 9050 4600 0    50   ~ 0
+SWDIO
+Text Label 9050 4700 0    50   ~ 0
+SWO
+$Sheet
+S 1550 5750 2350 900
+U 62053103
+F0 "microprocesor" 50
+F1 "microprocesor.sch" 50
+F2 "NTC" I R 3900 6050 50
+F3 "CURRENT" I R 3900 6200 50
+F4 "DAC" I R 3900 6400 50
+F5 "DIGITAL_T" I R 3900 5800 50
+F6 "SWDIO" I L 1550 5800 50
+F7 "SWDCLK" I L 1550 6100 50
+F8 "SDA" I L 1550 6350 50
+F9 "SCL" I L 1550 6200 50
+F10 "SWO" I L 1550 5950 50
+F11 "ANALOG_T" I R 3900 6500 50
+F12 "NRST" I R 3900 5900 50
+$EndSheet
+Wire Wire Line
+	4150 5800 3900 5800
+Wire Wire Line
+	4100 5900 3900 5900
+Wire Wire Line
+	4050 6050 3900 6050
+Wire Wire Line
+	4050 6200 3900 6200
+Wire Wire Line
+	4050 6400 3900 6400
+Wire Wire Line
+	4050 6500 3900 6500
+Text Label 4150 5800 0    50   ~ 0
+DIGITAL_T
+Text Label 4100 5900 0    50   ~ 0
+NRST
+Text Label 4050 6050 0    50   ~ 0
+NTC
+Text Label 4050 6200 0    50   ~ 0
+CURRENT
+Text Label 4050 6400 0    50   ~ 0
+DAC
+Text Label 4050 6500 0    50   ~ 0
+ANALOG_T
+Wire Wire Line
+	1350 5800 1550 5800
+Wire Wire Line
+	1350 5950 1550 5950
+Wire Wire Line
+	1350 6100 1550 6100
+Wire Wire Line
+	1350 6200 1550 6200
+Wire Wire Line
+	1350 6350 1550 6350
+Text Label 1350 5800 2    50   ~ 0
+SWDIO
+Text Label 1350 5950 2    50   ~ 0
+SWO
+Text Label 1350 6100 2    50   ~ 0
+SWDCLK
+Text Label 1350 6200 2    50   ~ 0
+SCL
+Text Label 1350 6350 2    50   ~ 0
+SDA
+$Sheet
+S 1650 1750 2550 1150
+U 6205B1FA
+F0 "BIAS" 50
+F1 "BIAS.sch" 50
+F2 "CURRENT" I R 4200 2050 50
+F3 "BIAS" I R 4200 2200 50
+F4 "DAC" I R 4200 2350 50
+$EndSheet
+Wire Wire Line
+	4350 2050 4200 2050
+Wire Wire Line
+	4400 2200 4200 2200
+Wire Wire Line
+	4400 2350 4200 2350
+Text Label 4350 2050 0    50   ~ 0
+CURRENT
+Text Label 4400 2200 0    50   ~ 0
+BIAS
+Text Label 4400 2350 0    50   ~ 0
+DAC
 $EndSCHEMATC

Commit message: Add files via upload
Connections:
- net +3V3 renamed +3.3V
Changed lines of the file:
@@
 Comment4 ""
 $EndDescr
-$Comp
-L power:GND #PWR02
-U 1 1 61E96DC1
-P 8450 1550
-F 0 "#PWR02" H 8450 1300 50  0001 C CNN
-F 1 "GND" V 8455 1422 50  0000 R CNN
-F 2 "" H 8450 1550 50  0001 C CNN
-F 3 "" H 8450 1550 50  0001 C CNN
-	1    8450 1550
-	0    -1   -1   0
-$EndComp
 Wire Wire Line
 	8250 1550 8450 1550
-$Comp
-L power:GND #PWR09
-U 1 1 61E9BAA5
-P 8650 1650
-F 0 "#PWR09" H 8650 1400 50  0001 C CNN
-F 1 "GND" V 8655 1522 50  0000 R CNN
-F 2 "" H 8650 1650 50  0001 C CNN
-F 3 "" H 8650 1650 50  0001 C CNN
-	1    8650 1650
-	0    -1   -1   0
-$EndComp
 Wire Wire Line
 	8250 1650 8650 1650
-$Comp
-L power:+5V #PWR05
-U 1 1 61EA08F2
-P 8550 1750
-F 0 "#PWR05" H 8550 1600 50  0001 C CNN
-F 1 "+5V" V 8565 1878 50  0000 L CNN
-F 2 "" H 8550 1750 50  0001 C CNN
-F 3 "" H 8550 1750 50  0001 C CNN
-	1    8550 1750
-	0    1    1    0
-$EndComp
 Wire Wire Line
 	8250 1750 8550 1750
-$Comp
-L power:GND #PWR03
-U 1 1 61EAA705
-P 8450 1850
-F 0 "#PWR03" H 8450 1600 50  0001 C CNN
-F 1 "GND" V 8455 1722 50  0000 R CNN
-F 2 "" H 8450 1850 50  0001 C CNN
-F 3 "" H 8450 1850 50  0001 C CNN
-	1    8450 1850
-	0    -1   -1   0
-$EndComp
 Wire Wire Line
 	8250 1850 8450 1850
@@
 Wire Wire Line
 	8550 2250 8250 2250
-$Comp
-L power:+3.3V #PWR06
-U 1 1 61EC92B3
-P 8550 2250
-F 0 "#PWR06" H 8550 2100 50  0001 C CNN
-F 1 "+3.3V" V 8565 2378 50  0000 L CNN
-F 2 "" H 8550 2250 50  0001 C CNN
-F 3 "" H 8550 2250 50  0001 C CNN
-	1    8550 2250
-	0    1    1    0
-$EndComp
 Wire Wire Line
 	8350 2350 8250 2350
-$Comp
-L power:GND #PWR01
-U 1 1 61ED4863
-P 8350 2350
-F 0 "#PWR01" H 8350 2100 50  0001 C CNN
-F 1 "GND" V 8355 2222 50  0000 R CNN
-F 2 "" H 8350 2350 50  0001 C CNN
-F 3 "" H 8350 2350 50  0001 C CNN
-	1    8350 2350
-	0    -1   -1   0
-$EndComp
 Wire Wire Line
 	8800 2450 8250 2450
@@
 	1    0    0    -1
 $EndComp
-$Comp
-L power:GND #PWR?
-U 1 1 61F1BCDB
-P 8450 5300
-AR Path="/61E803D7/61F1BCDB" Ref="#PWR?"  Part="1"
-AR Path="/61F1BCDB" Ref="#PWR04"  Part="1"
-F 0 "#PWR04" H 8450 5050 50  0001 C CNN
-F 1 "GND" H 8455 5127 50  0000 C CNN
-F 2 "" H 8450 5300 50  0001 C CNN
-F 3 "" H 8450 5300 50  0001 C CNN
-	1    8450 5300
-	1    0    0    -1
-$EndComp
-$Comp
-L power:GND #PWR?
-U 1 1 61F1BCE1
-P 8600 5300
-AR Path="/61E803D7/61F1BCE1" Ref="#PWR?"  Part="1"
-AR Path="/61F1BCE1" Ref="#PWR08"  Part="1"
-F 0 "#PWR08" H 8600 5050 50  0001 C CNN
-F 1 "GND" H 8605 5127 50  0000 C CNN
-F 2 "" H 8600 5300 50  0001 C CNN
-F 3 "" H 8600 5300 50  0001 C CNN
-	1    8600 5300
-	1    0    0    -1
-$EndComp
 Wire Wire Line
 	8550 5200 8600 5200
@@
 Wire Wire Line
 	8450 5200 8450 5300
-$Comp
-L power:+3.3V #PWR?
-U 1 1 61F1BCEA
-P 8550 3800
-AR Path="/61E803D7/61F1BCEA" Ref="#PWR?"  Part="1"
-AR Path="/61F1BCEA" Ref="#PWR07"  Part="1"
-F 0 "#PWR07" H 8550 3650 50  0001 C CNN
-F 1 "+3.3V" H 8565 3973 50  0000 C CNN
-F 2 "" H 8550 3800 50  0001 C CNN
-F 3 "" H 8550 3800 50  0001 C CNN
-	1    8550 3800
-	1    0    0    -1
-$EndComp
 Wire Wire Line
 	8550 3800 8550 4000
@@
 Wire Wire Line
 	8400 2750 8250 2750
-$Comp
-L power:GND #PWR0103
-U 1 1 61EFC12A
-P 8400 2750
-F 0 "#PWR0103" H 8400 2500 50  0001 C CNN
-F 1 "GND" V 8405 2622 50  0000 R CNN
-F 2 "" H 8400 2750 50  0001 C CNN
-F 3 "" H 8400 2750 50  0001 C CNN
-	1    8400 2750
-	0    -1   -1   0
-$EndComp
 $Comp
 L Connector:Conn_01x13_Male J1
@@
 F11 "ANALOG_T" I R 3900 6500 50
 F12 "NRST" I R 3900 5900 50
+F13 "GND" I L 1550 6500 50
+F14 "+3.3V" I R 3900 6600 50
+F15 "+5V" I L 1550 6600 50
 $EndSheet
 Wire Wire Line
@@
 F3 "BIAS" I R 4200 2200 50
 F4 "DAC" I R 4200 2350 50
+F5 "GND" I R 4200 2550 50
+F6 "+5V" I R 4200 2700 50
 $EndSheet
 Wire Wire Line
@@
 Text Label 4400 2350 0    50   ~ 0
 DAC
+Wire Wire Line
+	4450 2550 4200 2550
+Wire Wire Line
+	4450 2700 4200 2700
+Text Label 4450 2550 0    50   ~ 0
+GND
+Text Label 4450 2700 0    50   ~ 0
++5V
+Wire Wire Line
+	4100 6600 3900 6600
+Wire Wire Line
+	1350 6500 1550 6500
+Text Label 4100 6600 0    50   ~ 0
++3.3V
+Text Label 1350 6500 2    50   ~ 0
+GND
+Text Label 8400 2750 0    50   ~ 0
+GND
+Text Label 8350 2350 0    50   ~ 0
+GND
+Text Label 8550 2250 0    50   ~ 0
++3.3V
+Text Label 8450 1550 0    50   ~ 0
+GND
+Text Label 8650 1650 0    50   ~ 0
+GND
+Text Label 8550 1750 0    50   ~ 0
++5V
+Text Label 8450 1850 0    50   ~ 0
+GND
+Text Label 8600 5300 3    50   ~ 0
+GND
+Text Label 8450 5300 3    50   ~ 0
+GND
+Text Label 8550 3800 1    50   ~ 0
++3.3V
+Wire Wire Line
+	1350 6600 1550 6600
+Text Label 1350 6600 2    50   ~ 0
++5V
 $EndSCHEMATC

Commit message: Add files via upload
Changed lines of the file:
@@
 F5 "GND" I R 4200 2550 50
 F6 "+5V" I R 4200 2700 50
+F7 "+3.3V" I R 4200 1850 50
 $EndSheet
 Wire Wire Line
@@
 Text Label 1350 6600 2    50   ~ 0
 +5V
+Wire Wire Line
+	4400 1850 4200 1850
+Text Label 4400 1850 0    50   ~ 0
++3.3V
 $EndSCHEMATC
